File: BIRDS-X-PCB/BIRDS-X-PCB.kicad_pcb (KiCad board)
At the start: 2 copper layers, 85 x 85 mm, 77 parts, among them J101 LPC-50M2LG, J102 Conn_02x04_Odd_Even, J201 Conn_01x02, J202 Conn_01x02, J203 Conn_01x02, J401 Conn_02x04_Odd_Even, J402 Conn_01x08, Q201 SI1470DH, Q202 SI1470DH, Q401 BSS138, Q402 BSS138, SW401 SW_Push, U201 LTC4361-X, U202 LTC4361-X, U203 0.1S7B_3UP, U301 VT01, U302 VT01, U303 VT01, U304 VT01, U305 TL974IPWR, U306 ADG734, U307 LM335DT, U308 LM334M, U401 STM32G031K8Tx, U402 MTT4B-Mini, U403 MT29F2G01ABAGDWB-IT-G_TR, Y401 ECS-2520SMV-080-FN-TR

Commit message: Finish layout
Parts:
- added D401: LED, LED_SMD:LED_1206_3216Metric_Pad1.42x1.75mm_HandSolder, F.Cu at (102.7, 120.8)
- added J403: Conn_01x02, Connector_PinHeader_2.54mm:PinHeader_1x02_P2.54mm_Vertical, F.Cu at (103.5, 60.3)
- added J404: MHDR2X5, Connector_PinHeader_1.27mm:PinHeader_2x05_P1.27mm_Vertical_SMD, F.Cu at (97.1, 62.2)
- added R410: R, Resistor_SMD:R_0805_2012Metric_Pad1.20x1.40mm_HandSolder, F.Cu at (107.7, 120.8)
- added TP301: TestPoint, TestPoint:TestPoint_Pad_D2.0mm, F.Cu at (120.0, 54.0)
- C201, C202, C203, C204, C401, C402, C403, C404, C405, C406, C407, C408: footprint Capacitor_SMD:C_1206_3216Metric_Pad1.33x1.80mm_HandSolder -> Capacitor_SMD:C_0805_2012Metric_Pad1.18x1.45mm_HandSolder
- J401: value Conn_02x04_Odd_Even -> Conn_01x04; footprint Connector_PinSocket_2.54mm:PinSocket_2x04_P2.54mm_Vertical -> Connector_PinHeader_2.54mm:PinHeader_1x04_P2.54mm_Vertical
- R203, R204, R205, R401, R402, R403, R404, R405, R406, R407, R408, R409: footprint Resistor_SMD:R_1206_3216Metric_Pad1.30x1.75mm_HandSolder -> Resistor_SMD:R_0805_2012Metric_Pad1.20x1.40mm_HandSolder
- R301: renamed from R303; footprint Resistor_SMD:R_1206_3216Metric_Pad1.30x1.75mm_HandSolder -> Resistor_SMD:R_0805_2012Metric_Pad1.20x1.40mm_HandSolder
- R302: renamed from R2; footprint Resistor_SMD:R_1206_3216Metric -> Resistor_SMD:R_0805_2012Metric_Pad1.20x1.40mm_HandSolder
- R303: renamed from R1; footprint Resistor_SMD:R_1206_3216Metric -> Resistor_SMD:R_0805_2012Metric_Pad1.20x1.40mm_HandSolder
- R304: renamed from R3; footprint Resistor_SMD:R_1206_3216Metric -> Resistor_SMD:R_0805_2012Metric_Pad1.20x1.40mm_HandSolder
- R305: renamed from R4; footprint Resistor_SMD:R_1206_3216Metric -> Resistor_SMD:R_0805_2012Metric_Pad1.20x1.40mm_HandSolder
- R306: renamed from R5; footprint Resistor_SMD:R_1206_3216Metric -> Resistor_SMD:R_0805_2012Metric_Pad1.20x1.40mm_HandSolder
- R307: renamed from R6; footprint Resistor_SMD:R_1206_3216Metric -> Resistor_SMD:R_0805_2012Metric_Pad1.20x1.40mm_HandSolder
- R308: renamed from R7; footprint Resistor_SMD:R_1206_3216Metric -> Resistor_SMD:R_0805_2012Metric_Pad1.20x1.40mm_HandSolder
- R309: renamed from R8; footprint Resistor_SMD:R_1206_3216Metric -> Resistor_SMD:R_0805_2012Metric_Pad1.20x1.40mm_HandSolder
- R310: renamed from R9; footprint Resistor_SMD:R_1206_3216Metric -> Resistor_SMD:R_0805_2012Metric_Pad1.20x1.40mm_HandSolder
- R311: renamed from R10; footprint Resistor_SMD:R_1206_3216Metric -> Resistor_SMD:R_0805_2012Metric_Pad1.20x1.40mm_HandSolder
- TP401: footprint TestPoint:TestPoint_Pad_D2.5mm -> TestPoint:TestPoint_Pad_D2.0mm
- U201, U202: value LTC4361-X -> LTC4361-2
- U301, U302, U303, U304: value VT01 -> VT03; footprint Package_SO:SO-6_4.4x3.6mm_P1.27mm -> Package_TO_SOT_SMD:SOT-23-6_Handsoldering
- U402: footprint BIRDS-X_Footprints_Lib:MTT4B-Mini -> BIRDS-X_Footprints_Lib:MTT4B-Mini_CanUp
- moved C403 142.3 mm to (89.1, 79.4), turned to 180 degrees
- moved C402 142.3 mm to (89.1, 76.8), turned to 180 degrees
- moved C401 142.3 mm to (89.1, 85.1), turned to 180 degrees
- moved C404 141.5 mm to (91.4, 68.2), turned to 90 degrees
- moved D201 139.1 mm to (102.5, 110.2)
- moved D202 139.1 mm to (102.5, 113.6)
- moved D203 139.1 mm to (102.5, 116.9)
- moved C203 135.1 mm to (94.3, 119.5)
- moved C204 130.8 mm to (94.7, 96.6)
- moved R403 127.4 mm to (87.3, 71.1)
- moved J203 125.1 mm to (114.4, 120.1), turned to 90 degrees
- moved U301 124.6 mm to (96.4, 53.7)
- moved C202 124.4 mm to (102.3, 102.0), turned to -90 degrees
- moved U304 123.1 mm to (86.3, 120.3)
- moved C406 121.9 mm to (115.4, 81.3)
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Connections:
- C401 pad 1: Net-(U401-PF2) -> ST_RST
- D201 pad 1: Net-(D201-K) -> GND
- D201 pad 2: GND -> Net-(D201-A)
- D202 pad 1: Net-(D202-K) -> GND
- D202 pad 2: GND -> Net-(D202-A)
- D203 pad 1: Net-(D203-K) -> GND
- D203 pad 2: GND -> Net-(D203-A)
- J101 pad 1: PROG_DBG_1 -> ST_SWDIO
- J101 pad 2: PROG_DBG_2 -> BOOT0
- J101 pad 3: PROG_DBG_3 -> ST_RST
- J401 pad 2: GND -> Net-(J401-Pin_2)
- J401 pad 3: Net-(J401-Pin_3) -> +5V
- J401 pad 4: Net-(J401-Pin_3) -> Net-(J401-Pin_4)
- JP403 pad 1: Net-(J401-Pin_3) -> Net-(J401-Pin_2)
- JP404 pad 1: Net-(J401-Pin_7) -> Net-(J401-Pin_4)
- Q401 pad 3: Net-(J401-Pin_3) -> Net-(J401-Pin_2)
- Q402 pad 3: Net-(J401-Pin_7) -> Net-(J401-Pin_4)
- R203 pad 2: Net-(D201-K) -> Net-(D201-A)
- R204 pad 2: Net-(D202-K) -> Net-(D202-A)
- R205 pad 2: Net-(D203-K) -> Net-(D203-A)
- R405 pad 2: Net-(J401-Pin_3) -> Net-(J401-Pin_2)
- R406 pad 2: Net-(J401-Pin_7) -> Net-(J401-Pin_4)
- SW401 pad 2: Net-(U401-PF2) -> ST_RST
- U301 pad 3: GND -> unconnected-(U301-NC-Pad3)
- U301 pad 5: GND -> unconnected-(U301-NC-Pad5)
- U302 pad 3: GND -> unconnected-(U302-NC-Pad3)
- U302 pad 5: GND -> unconnected-(U302-NC-Pad5)
- U303 pad 3: GND -> unconnected-(U303-NC-Pad3)
- U303 pad 5: GND -> unconnected-(U303-NC-Pad5)
- U304 pad 3: GND -> unconnected-(U304-NC-Pad3)
- U304 pad 5: GND -> unconnected-(U304-NC-Pad5)
- U308 pad 4: +5V -> +12V
- U401 pad 22: unconnected-(U401-PA11/PA9-Pad22) -> Net-(U401-PA11/PA9)
- U401 pad 23: unconnected-(U401-PA12/PA10-Pad23) -> Net-(J403-Pin_1)
- U401 pad 24: unconnected-(U401-PA13-Pad24) -> ST_SWDIO
- U401 pad 26: unconnected-(U401-PA15-Pad26) -> Net-(J403-Pin_2)
- U401 pad 6: Net-(U401-PF2) -> ST_RST
- U402 pad J2-2: Net-(J401-Pin_3) -> Net-(J401-Pin_2)
- U402 pad J2-4: Net-(J401-Pin_7) -> Net-(J401-Pin_4)

Commit message: Update footprint
Parts:
- moved JP201 0.89 mm to (114.3, 98.4)
- moved Y401 0.64 mm to (90.7, 72.7)
Changed lines of the file:
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@@
   )
   (footprint "lib:OSC_ECS-2520SMV-080-FN-TR" (layer "F.Cu")
-    (at 90.715 72.1 -90)
+    (at 90.715 72.735 -90)
     (property "Sheetfile" "MicrocontrollerSheet.kicad_sch")
     (property "Sheetname" "MicrocontrollerSheet")
     (attr smd)
-    (fp_text reference "Y401" (at -0.762633 -1.807066 90) (layer "F.SilkS")
-        (effects (font (size 0.320686 0.320686) (thickness 0.15)))
-    )
-    (fp_text value "ECS-2520SMV-080-FN-TR" (at 3.336563 1.91958 90) (layer "F.Fab")
+    (fp_text reference "Y401" (at 0 -2 -90) (layer "F.SilkS")
+        (effects (font (size 1 1) (thickness 0.15)))
+    )
+    (fp_text value "ECS-2520SMV-080-FN-TR" (at 3.336563 1.91958 -90) (layer "F.Fab")
         (effects (font (size 0.320631 0.320631) (thickness 0.15)))
     )
@@
     (fp_line (start -0.221 1) (end 0.221 1)
       (stroke (width 0.127) (type solid)) (layer "F.SilkS"))
-    (fp_circle (center -1.9 0.85) (end -1.8 0.85)
-      (stroke (width 0.2) (type solid)) (fill none) (layer "F.SilkS"))
+    (fp_circle (center -2 0.85) (end -1.7 0.85)
+      (stroke (width 0.2) (type solid)) (fill solid) (layer "F.SilkS"))
     (fp_line (start -1.625 -1.375) (end 1.625 -1.375)
       (stroke (width 0.05) (type solid)) (layer "F.CrtYd"))
@@
   )
   (footprint "Jumper:SolderJumper-2_P1.3mm_Open_RoundedPad1.0x1.5mm" (layer "F.Cu")
-    (at 115.015 97.92)
+    (at 114.285 98.425)
     (descr "SMD Solder Jumper, 1x1.5mm, rounded Pads, 0.3mm gap, open")
     (tags "solder jumper open")

Commit message: Do some routing
Parts:
- added D301: 1N457, Diode_THT:D_DO-35_SOD27_P7.62mm_Horizontal, F.Cu at (101.6, 52.2)
- added JP301: Jumper_2_Open, Connector_PinHeader_2.54mm:PinHeader_1x02_P2.54mm_Vertical, F.Cu at (106.5, 52.8)
- R302: value 10k -> 11k
- R303: value 390k -> 110k
- moved C203 31.5 mm to (62.8, 118.5)
- moved C201 31.5 mm to (82.3, 101.6)
- moved C202 31.5 mm to (70.8, 101.0)
- moved C404 31.5 mm to (59.9, 67.2)
- moved C405 31.5 mm to (83.9, 77.7)
- moved C406 31.5 mm to (83.9, 80.3)
- moved C407 31.5 mm to (103.8, 85.8)
- moved C408 31.5 mm to (103.8, 89.2)
- moved D201 31.5 mm to (71.0, 109.2)
- moved D202 31.5 mm to (71.0, 112.6)
- moved D203 31.5 mm to (71.0, 115.9)
- moved D401 31.5 mm to (71.2, 119.8)
- moved H101 31.5 mm to (57.0, 57.7)
- moved H102 31.5 mm to (127.0, 57.7)
- moved H103 31.5 mm to (57.0, 127.7)
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Connections:
- R302 pad 2: Net-(R302-Pad2) -> Net-(D301-A)
- R303 pad 1: Net-(R302-Pad2) -> Net-(R302-Pad1)
- R303 pad 2: Net-(R303-Pad2) -> Net-(D301-K)
- U306 pad 14: Net-(R303-Pad2) -> Net-(JP301-B)
- U306 pad 17: Net-(R303-Pad2) -> Net-(JP301-B)
- U306 pad 4: Net-(R303-Pad2) -> Net-(JP301-B)
- U306 pad 7: Net-(R303-Pad2) -> Net-(JP301-B)
- U308 pad 2: Net-(R303-Pad2) -> Net-(D301-A)
- U308 pad 3: Net-(R303-Pad2) -> Net-(D301-A)
- U308 pad 6: Net-(R303-Pad2) -> Net-(D301-A)
- U308 pad 7: Net-(R303-Pad2) -> Net-(D301-A)
Routing:
- net +3V3: track 0.00 -> 130.6 mm, vias 0 -> 14
- net +5V: track 0.00 -> 102.0 mm, vias 0 -> 9
- net ST_RST: track 0.00 -> 87.0 mm, vias 0 -> 3
- net BOOT0: track 0.00 -> 82.1 mm, vias 0 -> 4
- net ST_SWDIO: track 0.00 -> 71.1 mm, vias 0 -> 3
- net UART_TX_JASPER_TO_BOSS: track 0.00 -> 67.8 mm, vias 0 -> 2
- net UART_RX_BOSS_TO_JASPER: track 0.00 -> 67.0 mm, vias 0 -> 2
- net Net-(JP404-B): track 0.00 -> 52.1 mm, vias 0 -> 4
- net Net-(U401-PA11/PA9): track 0.00 -> 50.2 mm, vias 0 -> 2
- net +12V: track 0.00 -> 42.3 mm, vias 0 -> 4
- net RFET_EN1: track 0.00 -> 38.2 mm, vias 0 -> 1
- net DIO2_5V_EN_FROM_BOSS: track 0.00 -> 35.9 mm, vias 0 -> 2
- net Net-(J401-Pin_4): track 0.00 -> 35.2 mm, vias 0 -> 1
- net SUP_5V0: track 0.00 -> 33.3 mm, vias 0 -> 1
- net Net-(J401-Pin_2): track 0.00 -> 32.9 mm, vias 0 -> 4
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- added copper zone on B.Cu, net GND
- added copper zone on F.Cu, net GND
Other:
- outline, holes or cut-outs redrawn
- board text added: "(0,0) is (50,50)"
- board text removed: "(0,0) is (81,51)"

Commit message: Route more, move MCU
Parts:
- moved D301 47.4 mm to (70.5, 88.1), turned to 90 degrees
- moved R302 30.5 mm to (62.4, 87.5), turned to 90 degrees
- moved R403 30.5 mm to (86.2, 71.3), turned to -90 degrees
- moved C404 30.1 mm to (88.9, 75.5), turned to 0 degrees
- moved U308 30.0 mm to (64.0, 82.6)
- moved J102 29.3 mm to (75.0, 89.2), turned to 90 degrees
- moved J403 27.5 mm to (95.7, 73.2), turned to 90 degrees
- moved Y401 25.3 mm to (84.3, 74.8), turned to 180 degrees
- moved R303 25.2 mm to (66.2, 87.5), turned to 90 degrees
- moved C402 22.0 mm to (79.5, 73.7), turned to 90 degrees
- moved C405 21.4 mm to (63.7, 70.5)
- moved C406 21.4 mm to (63.7, 73.0)
- moved R409 21.0 mm to (54.9, 66.9)
- moved U403 21.0 mm to (57.0, 73.5)
- moved R408 21.0 mm to (58.7, 66.8)
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Routing:
- net ST_RST: track 87.0 -> 0.00 mm, vias 3 -> 0
- net BOOT0: track 82.1 -> 0.00 mm, vias 4 -> 0
- net +12V: track 42.3 -> 115.4 mm, vias 4 -> 9
- net ST_SWDIO: track 71.1 -> 0.00 mm, vias 3 -> 0
- net UART_TX_JASPER_TO_BOSS: track 67.8 -> 0.00 mm, vias 2 -> 0
- net UART_RX_BOSS_TO_JASPER: track 67.0 -> 0.00 mm, vias 2 -> 0
- net +3V3: track 130.6 -> 197.2 mm, vias 14 -> 19
- net RFET_OUT4: track 0.00 -> 60.0 mm, vias 0 -> 6
- net RFET_OUT3: track 0.00 -> 54.5 mm, vias 0 -> 4
- net Net-(U401-PA11/PA9): track 50.2 -> 0.00 mm, vias 2 -> 0
- net Net-(JP404-B): track 52.1 -> 9.36 mm, vias 4 -> 2
- net RFET_OUT1: track 0.00 -> 41.2 mm, vias 0 -> 6
- net RFET_OUT2: track 0.00 -> 40.4 mm, vias 0 -> 6
- net RFET_EN1: track 38.2 -> 0.00 mm, vias 1 -> 0
- net MEM_MOSI: track 16.1 -> 0.00 mm, vias 2 -> 0
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
Commit message: PCB update
Parts:
- moved R302 36.7 mm to (82.5, 56.8), turned to 180 degrees
- moved R408 35.9 mm to (83.8, 92.5), turned to 90 degrees
- moved R303 31.9 mm to (82.5, 60.0), turned to 180 degrees
- moved U308 30.6 mm to (89.3, 65.3)
- moved D301 29.1 mm to (93.1, 69.7), turned to 180 degrees
- moved R409 26.0 mm to (67.8, 89.5)
- moved U403 24.7 mm to (75.4, 90.0)
- moved C406 24.4 mm to (83.7, 87.0), turned to 90 degrees
- moved C405 24.0 mm to (81.2, 87.0), turned to 90 degrees
- moved TP401 22.5 mm to (60.8, 72.2), turned to 0 degrees
- moved J102 22.1 mm to (56.3, 77.3), turned to 0 degrees
- moved R402 19.5 mm to (88.8, 74.5), turned to -90 degrees
- moved R401 17.6 mm to (88.8, 78.2), turned to 90 degrees
- moved JP401 16.2 mm to (84.0, 81.0)
- moved J402 12.5 mm to (53.7, 92.5)
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Routing:
- net +3V3: track 197.2 -> 51.8 mm, vias 19 -> 7
- net Net-(U304-SOURCE_BULK): track 0.00 -> 133.1 mm
- net Net-(U303-SOURCE_BULK): track 0.00 -> 90.0 mm
- net RFET_EN4: track 0.00 -> 86.7 mm, vias 0 -> 4
- net +12V: track 115.4 -> 38.9 mm, vias 9 -> 3
- net RFET_EN3: track 0.00 -> 76.0 mm, vias 0 -> 4
- net RFET_EN1: track 0.00 -> 71.2 mm, vias 0 -> 6
- net RFET_EN2: track 0.00 -> 68.8 mm, vias 0 -> 2
- net MEM_CLK: track 0.00 -> 56.2 mm, vias 0 -> 2
- net MEM_MOSI: track 0.00 -> 40.2 mm
- net RFET_OUT3: track 54.5 -> 93.4 mm, vias 4 -> 2
- net Net-(U301-SOURCE_BULK): track 0.00 -> 36.1 mm
- net RFET_OUT4: track 60.0 -> 93.7 mm, vias 6 -> 2
- net MEM_MISO: track 0.00 -> 30.6 mm
- net RFET_OUT1: track 41.2 -> 71.0 mm, vias 6 -> 2
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