File: BIRDS-X-PCB/RF_System.kicad_sch (KiCad schematic)
At the start: 23 parts, among them J501 60611002111501, Q501 BC847, U503 DRA818V

Commit message: Schematic re-work (esp. RADFET fixes)
Parts:
- renumbered J501 to J401, Q501 to Q401, U503 to U401
Changed lines of the file:
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@@
         )
         (path "/c2796b15-795a-4d6e-ad4b-0ba87ded4bc9/245c031a-1c72-4f7a-bf07-271990525459"
-          (reference "C504") (unit 1)
+          (reference "C403") (unit 1)
         )
       )
@@
         )
         (path "/c2796b15-795a-4d6e-ad4b-0ba87ded4bc9/245c031a-1c72-4f7a-bf07-271990525459"
-          (reference "C512") (unit 1)
+          (reference "C407") (unit 1)
         )
       )
@@
   (symbol (lib_id "BIRDS-X_Symbols_Lib:DRA818V") (at 222.25 57.15 0) (unit 1)
     (in_bom yes) (on_board yes) (dnp no) (fields_autoplaced)
-    (property "Reference" "U503" (at 222.25 39.37 0)
+    (property "Reference" "U401" (at 222.25 39.37 0)
       (effects (font (size 1.27 1.27)))
     )
@@
       (project "BIRDS-X-PCB"
         (path "/c2796b15-795a-4d6e-ad4b-0ba87ded4bc9/245c031a-1c72-4f7a-bf07-271990525459"
-          (reference "U503") (unit 1)
+          (reference "U401") (unit 1)
         )
       )
@@
         )
         (path "/c2796b15-795a-4d6e-ad4b-0ba87ded4bc9/245c031a-1c72-4f7a-bf07-271990525459"
-          (reference "C507") (unit 1)
+          (reference "C405") (unit 1)
         )
       )
@@
         )
         (path "/c2796b15-795a-4d6e-ad4b-0ba87ded4bc9/245c031a-1c72-4f7a-bf07-271990525459"
-          (reference "#PWR0506") (unit 1)
+          (reference "#PWR0402") (unit 1)
         )
       )
@@
         )
         (path "/c2796b15-795a-4d6e-ad4b-0ba87ded4bc9/245c031a-1c72-4f7a-bf07-271990525459"
-          (reference "C502") (unit 1)
+          (reference "C404") (unit 1)
         )
       )
@@
         )
         (path "/c2796b15-795a-4d6e-ad4b-0ba87ded4bc9/245c031a-1c72-4f7a-bf07-271990525459"
-          (reference "#PWR0502") (unit 1)
+          (reference "#PWR0404") (unit 1)
         )
       )
@@
         )
         (path "/c2796b15-795a-4d6e-ad4b-0ba87ded4bc9/245c031a-1c72-4f7a-bf07-271990525459"
-          (reference "R512") (unit 1)
+          (reference "R413") (unit 1)
         )
       )
@@
         )
         (path "/c2796b15-795a-4d6e-ad4b-0ba87ded4bc9/245c031a-1c72-4f7a-bf07-271990525459"
-          (reference "R513") (unit 1)
+          (reference "R402") (unit 1)
         )
       )
@@
         )
         (path "/c2796b15-795a-4d6e-ad4b-0ba87ded4bc9/245c031a-1c72-4f7a-bf07-271990525459"
-          (reference "#PWR0501") (unit 1)
+          (reference "#PWR0401") (unit 1)
         )
       )
@@
         )
         (path "/c2796b15-795a-4d6e-ad4b-0ba87ded4bc9/245c031a-1c72-4f7a-bf07-271990525459"
-          (reference "R502") (unit 1)
+          (reference "R404") (unit 1)
         )
       )
@@
       (project "BIRDS-X-PCB"
         (path "/c2796b15-795a-4d6e-ad4b-0ba87ded4bc9/245c031a-1c72-4f7a-bf07-271990525459"
-          (reference "#PWR0517") (unit 1)
+          (reference "#PWR0409") (unit 1)
         )
       )
@@
   (symbol (lib_id "Transistor_BJT:BC847") (at 73.66 77.47 0) (unit 1)
     (in_bom yes) (on_board yes) (dnp no) (fields_autoplaced)
-    (property "Reference" "Q501" (at 78.74 76.2 0)
+    (property "Reference" "Q401" (at 78.74 76.2 0)
       (effects (font (size 1.27 1.27)) (justify left))
     )
@@
       (project "BIRDS-X-PCB"
         (path "/c2796b15-795a-4d6e-ad4b-0ba87ded4bc9/245c031a-1c72-4f7a-bf07-271990525459"
-          (reference "Q501") (unit 1)
+          (reference "Q401") (unit 1)
         )
       )
@@
         )
         (path "/c2796b15-795a-4d6e-ad4b-0ba87ded4bc9/245c031a-1c72-4f7a-bf07-271990525459"
-          (reference "R511") (unit 1)
+          (reference "R403") (unit 1)
         )
       )
@@
         )
         (path "/c2796b15-795a-4d6e-ad4b-0ba87ded4bc9/245c031a-1c72-4f7a-bf07-271990525459"
-          (reference "R503") (unit 1)
+          (reference "R407") (unit 1)
         )
       )
@@
         )
         (path "/c2796b15-795a-4d6e-ad4b-0ba87ded4bc9/245c031a-1c72-4f7a-bf07-271990525459"
-          (reference "#PWR0505") (unit 1)
+          (reference "#PWR0406") (unit 1)
         )
       )
@@
         )
         (path "/c2796b15-795a-4d6e-ad4b-0ba87ded4bc9/245c031a-1c72-4f7a-bf07-271990525459"
-          (reference "R505") (unit 1)
+          (reference "R409") (unit 1)
         )
       )
@@
         )
         (path "/c2796b15-795a-4d6e-ad4b-0ba87ded4bc9/245c031a-1c72-4f7a-bf07-271990525459"
-          (reference "C503") (unit 1)
+          (reference "C406") (unit 1)
         )
       )
@@
         )
         (path "/c2796b15-795a-4d6e-ad4b-0ba87ded4bc9/245c031a-1c72-4f7a-bf07-271990525459"
-          (reference "R504") (unit 1)
+          (reference "R408") (unit 1)
         )
       )
@@
         )
         (path "/c2796b15-795a-4d6e-ad4b-0ba87ded4bc9/245c031a-1c72-4f7a-bf07-271990525459"
-          (reference "R510") (unit 1)
+          (reference "R406") (unit 1)
         )
       )
@@
         )
         (path "/c2796b15-795a-4d6e-ad4b-0ba87ded4bc9/245c031a-1c72-4f7a-bf07-271990525459"
-          (reference "C501") (unit 1)
+          (reference "C402") (unit 1)
         )
       )
@@
         )
         (path "/c2796b15-795a-4d6e-ad4b-0ba87ded4bc9/245c031a-1c72-4f7a-bf07-271990525459"
-          (reference "#PWR0504") (unit 1)
+          (reference "#PWR0403") (unit 1)
         )
       )
@@
         )
         (path "/c2796b15-795a-4d6e-ad4b-0ba87ded4bc9/245c031a-1c72-4f7a-bf07-271990525459"
-          (reference "#PWR0503") (unit 1)
+          (reference "#PWR0405") (unit 1)
         )
       )
@@
       (project "BIRDS-X-PCB"
         (path "/c2796b15-795a-4d6e-ad4b-0ba87ded4bc9/245c031a-1c72-4f7a-bf07-271990525459"
-          (reference "#PWR0518") (unit 1)
+          (reference "#PWR0411") (unit 1)
         )
       )
@@
         )
         (path "/c2796b15-795a-4d6e-ad4b-0ba87ded4bc9/245c031a-1c72-4f7a-bf07-271990525459"
-          (reference "R508") (unit 1)
+          (reference "R411") (unit 1)
         )
       )
@@
         )
         (path "/c2796b15-795a-4d6e-ad4b-0ba87ded4bc9/245c031a-1c72-4f7a-bf07-271990525459"
-          (reference "R506") (unit 1)
+          (reference "R412") (unit 1)
         )
       )
@@
         )
         (path "/c2796b15-795a-4d6e-ad4b-0ba87ded4bc9/245c031a-1c72-4f7a-bf07-271990525459"
-          (reference "R509") (unit 1)
+          (reference "R405") (unit 1)
         )
       )
@@
         )
         (path "/c2796b15-795a-4d6e-ad4b-0ba87ded4bc9/245c031a-1c72-4f7a-bf07-271990525459"
-          (reference "R501") (unit 1)
+          (reference "R401") (unit 1)
         )
       )
@@
         )
         (path "/c2796b15-795a-4d6e-ad4b-0ba87ded4bc9/245c031a-1c72-4f7a-bf07-271990525459"
-          (reference "R507") (unit 1)
+          (reference "R410") (unit 1)
         )
       )
@@
   (symbol (lib_id "Connector:Conn_Coaxial") (at 223.52 81.28 0) (unit 1)
     (in_bom yes) (on_board yes) (dnp no)
-    (property "Reference" "J501" (at 220.98 74.93 0)
+    (property "Reference" "J401" (at 220.98 74.93 0)
       (effects (font (size 1.27 1.27)) (justify left))
     )
@@
       (project "BIRDS-X-PCB"
         (path "/c2796b15-795a-4d6e-ad4b-0ba87ded4bc9/245c031a-1c72-4f7a-bf07-271990525459"
-          (reference "J501") (unit 1)
+          (reference "J401") (unit 1)
         )
       )
@@
       (project "BIRDS-X-PCB"
         (path "/c2796b15-795a-4d6e-ad4b-0ba87ded4bc9/245c031a-1c72-4f7a-bf07-271990525459"
-          (reference "#PWR0519") (unit 1)
+          (reference "#PWR0407") (unit 1)
         )
       )
@@
         )
         (path "/c2796b15-795a-4d6e-ad4b-0ba87ded4bc9/245c031a-1c72-4f7a-bf07-271990525459"
-          (reference "C506") (unit 1)
+          (reference "C401") (unit 1)
         )
       )
@@
         )
         (path "/c2796b15-795a-4d6e-ad4b-0ba87ded4bc9/245c031a-1c72-4f7a-bf07-271990525459"
-          (reference "#PWR025") (unit 1)
+          (reference "#PWR0410") (unit 1)
         )
       )
@@
         )
         (path "/c2796b15-795a-4d6e-ad4b-0ba87ded4bc9/245c031a-1c72-4f7a-bf07-271990525459"
-          (reference "#PWR0520") (unit 1)
-        )
-      )
+          (reference "#PWR0408") (unit 1)
+        )
+      )
